Commit message: update gait & legs

File: src/robots/configs/victor_config/urdf/accessories.urdf.xacro (robot description, xacro)
@@ -12,10 +12,10 @@
 			min_angle="130"
 			max_angle="-130" >
-			<origin xyz="0.0 0.0 ${base_height / 2 + 0.04}" rpy="0 0 0"/>
+			<origin xyz="0.0 0.0 ${base_height / 2 + 0.06}" rpy="0 0 0"/>
 		</xacro:hokuyo_utm30lx>
 		<xacro:asus_camera
 			parent="${base_name}"
 			name="camera">
-			<origin xyz="${base_length / 1} 0.0 ${base_height / 2 + .01}" rpy="0 0 0"/>
+			<origin xyz="${base_length + .1} 0.0 ${base_height / 2 + .01}" rpy="0 0 0"/>
 		</xacro:asus_camera>
 	<gazebo>

File: src/robots/configs/victor_config/urdf/quadruped.urdf (robot description, URDF)
Before this commit: robot victor, 29 links, 28 joints
Joints:
- joint camera_joint: origin xyz=0.175 0.0 0.015 rpy=0 0 0 -> xyz=0.275 0.0 0.015 rpy=0 0 0
- joint hokuyo_joint: origin xyz=0.0 0.0 0.045 rpy=0 0 0 -> xyz=0.0 0.0 0.065 rpy=0 0 0

Commit message: removed camera

File: src/robots/configs/victor_config/urdf/accessories.urdf.xacro (robot description, xacro)
@@ -3,5 +3,5 @@
 	<xacro:macro name="accessories" params="base_name base_length base_height  " >
 		<xacro:include filename="$(find hector_sensors_description)/urdf/hokuyo_utm30lx.urdf.xacro" />
-		<xacro:include filename="$(find hector_sensors_description)/urdf/asus_camera.urdf.xacro" />
+		<!---<xacro:include filename="$(find hector_sensors_description)/urdf/asus_camera.urdf.xacro" /> -->
 		<xacro:hokuyo_utm30lx
 			name="hokuyo"
@@ -14,9 +14,9 @@
 			<origin xyz="0.0 0.0 ${base_height / 2 + 0.06}" rpy="0 0 0"/>
 		</xacro:hokuyo_utm30lx>
-		<xacro:asus_camera
+		<!--<xacro:asus_camera
 			parent="${base_name}"
 			name="camera">
 			<origin xyz="${base_length + .1} 0.0 ${base_height / 2 + .01}" rpy="0 0 0"/>
-		</xacro:asus_camera>
+		</xacro:asus_camera>-->
 	<gazebo>
 		<plugin name="imu_controller" filename="libhector_gazebo_ros_imu.so">

File: src/robots/configs/victor_config/urdf/quadruped.urdf (robot description, URDF)
Before this commit: robot victor, 29 links, 28 joints
Links:
- removed link camera_depth_frame
- removed link camera_depth_optical_frame
- removed link camera_link
- removed link camera_rgb_frame
- removed link camera_rgb_optical_frame
Joints:
- removed joint camera_depth_joint
- removed joint camera_depth_optical_joint
- removed joint camera_joint
- removed joint camera_rgb_joint
- removed joint camera_rgb_optical_joint
